File: 1_LED.sch (KiCad schematic (older format))
At the start: 8 parts

Commit message: All tasks were edited after feedback
Parts:
- added C3: 470 uF, symbol Device:C
- added R4: 100K, symbol Device:R
- R1: value 124 -> 130
- R2: value 175 -> 180
- R3: value 135 -> 330
Connections:
- wire segments 20 -> 25
Other:
- note added: "LED Voltage, V = 3.3 V\nLED Currect, I = 10 mA (brightness will be same, but LED life will be longer)\nResistor, R = U/I = 330 Om\n"
- moved on the sheet: C1, C2, DA1, R1, R2
Changed lines of the file:
@@
 $EndComp
 Wire Wire Line
-	2750 3350 2750 3400
+	2450 2750 2450 2800
 $Comp
 L power:GND #PWR?
 U 1 1 60786F64
-P 2000 3400
-F 0 "#PWR?" H 2000 3150 50  0001 C CNN
-F 1 "GND" H 2005 3227 50  0000 C CNN
-F 2 "" H 2000 3400 50  0001 C CNN
-F 3 "" H 2000 3400 50  0001 C CNN
-	1    2000 3400
+P 1900 3100
+F 0 "#PWR?" H 1900 2850 50  0001 C CNN
+F 1 "GND" H 1905 2927 50  0000 C CNN
+F 2 "" H 1900 3100 50  0001 C CNN
+F 3 "" H 1900 3100 50  0001 C CNN
+	1    1900 3100
 	1    0    0    -1
 $EndComp
@@
 L power:+5V #PWR?
 U 1 1 60787F59
-P 2000 3100
-F 0 "#PWR?" H 2000 2950 50  0001 C CNN
-F 1 "+5V" H 2015 3273 50  0000 C CNN
-F 2 "" H 2000 3100 50  0001 C CNN
-F 3 "" H 2000 3100 50  0001 C CNN
-	1    2000 3100
+P 1700 2500
+F 0 "#PWR?" H 1700 2350 50  0001 C CNN
+F 1 "+5V" H 1715 2673 50  0000 C CNN
+F 2 "" H 1700 2500 50  0001 C CNN
+F 3 "" H 1700 2500 50  0001 C CNN
+	1    1700 2500
 	1    0    0    -1
 $EndComp
 Wire Wire Line
-	3050 3100 3100 3100
-Wire Wire Line
-	4600 2550 4600 2700
-Text Label 3100 3050 0    50   ~ 0
+	2750 2500 2800 2500
+Text Label 2800 2450 0    50   ~ 0
 +3.3V
 $Comp
 L Device:CP1 C1
 U 1 1 6078E2D4
-P 2200 3250
-F 0 "C1" H 2315 3296 50  0000 L CNN
-F 1 "10 uF" H 2315 3205 50  0000 L CNN
-F 2 "" H 2200 3250 50  0001 C CNN
-F 3 "~" H 2200 3250 50  0001 C CNN
-	1    2200 3250
+P 1900 2650
+F 0 "C1" H 2015 2696 50  0000 L CNN
+F 1 "10 uF" H 2015 2605 50  0000 L CNN
+F 2 "" H 1900 2650 50  0001 C CNN
+F 3 "~" H 1900 2650 50  0001 C CNN
+	1    1900 2650
 	1    0    0    -1
 $EndComp
@@
 L Regulator_Linear:AMS1117 DA1
 U 1 1 60782483
-P 2750 3100
-F 0 "DA1" H 2750 3342 50  0000 C CNN
-F 1 "AMS1117" H 2750 3251 50  0000 C CNN
-F 2 "Package_TO_SOT_SMD:SOT-223-3_TabPin2" H 2750 3300 50  0001 C CNN
-F 3 "http://www.advanced-monolithic.com/pdf/ds1117.pdf" H 2850 2850 50  0001 C CNN
-	1    2750 3100
+P 2450 2500
+F 0 "DA1" H 2450 2742 50  0000 C CNN
+F 1 "AMS1117" H 2450 2651 50  0000 C CNN
+F 2 "Package_TO_SOT_SMD:SOT-223-3_TabPin2" H 2450 2700 50  0001 C CNN
+F 3 "http://www.advanced-monolithic.com/pdf/ds1117.pdf" H 2550 2250 50  0001 C CNN
+	1    2450 2500
 	1    0    0    -1
 $EndComp
-Connection ~ 2200 3100
+Connection ~ 1900 2500
 Wire Wire Line
-	2200 3100 2000 3100
+	1900 2500 1700 2500
 Wire Wire Line
-	2200 3400 2000 3400
-Wire Wire Line
-	2200 3100 2450 3100
+	1900 2500 2150 2500
 $Comp
 L Device:R R1
 U 1 1 607905E1
-P 3100 3250
-F 0 "R1" H 3170 3296 50  0000 L CNN
-F 1 "124" H 3170 3205 50  0000 L CNN
-F 2 "" V 3030 3250 50  0001 C CNN
-F 3 "~" H 3100 3250 50  0001 C CNN
-	1    3100 3250
+P 2800 2650
+F 0 "R1" H 2870 2696 50  0000 L CNN
+F 1 "130" H 2870 2605 50  0000 L CNN
+F 2 "" V 2730 2650 50  0001 C CNN
+F 3 "~" H 2800 2650 50  0001 C CNN
+	1    2800 2650
 	1    0    0    -1
 $EndComp
@@
 L Device:R R2
 U 1 1 60791220
-P 3100 3550
-F 0 "R2" H 3170 3596 50  0000 L CNN
-F 1 "175" H 3170 3505 50  0000 L CNN
-F 2 "" V 3030 3550 50  0001 C CNN
-F 3 "~" H 3100 3550 50  0001 C CNN
-	1    3100 3550
+P 2800 2950
+F 0 "R2" H 2870 2996 50  0000 L CNN
+F 1 "180" H 2870 2905 50  0000 L CNN
+F 2 "" V 2730 2950 50  0001 C CNN
+F 3 "~" H 2800 2950 50  0001 C CNN
+	1    2800 2950
 	1    0    0    -1
 $EndComp
 Wire Wire Line
-	3100 3400 2750 3400
-Connection ~ 3100 3400
-Connection ~ 2750 3400
+	2800 2800 2450 2800
+Connection ~ 2800 2800
+Connection ~ 2450 2800
 Wire Wire Line
-	2200 3400 2200 3700
-Wire Wire Line
-	2200 3700 3100 3700
-Connection ~ 2200 3400
+	1900 2800 1900 3100
 $Comp
 L Device:CP1 C2
 U 1 1 6079584F
-P 3600 3400
-F 0 "C2" H 3715 3446 50  0000 L CNN
-F 1 "22 uF" H 3715 3355 50  0000 L CNN
-F 2 "" H 3600 3400 50  0001 C CNN
-F 3 "~" H 3600 3400 50  0001 C CNN
-	1    3600 3400
+P 3200 2800
+F 0 "C2" H 3315 2846 50  0000 L CNN
+F 1 "22 uF" H 3315 2755 50  0000 L CNN
+F 2 "" H 3200 2800 50  0001 C CNN
+F 3 "~" H 3200 2800 50  0001 C CNN
+	1    3200 2800
 	1    0    0    -1
 $EndComp
 Wire Wire Line
-	3600 3550 3600 3700
+	2800 3100 3200 3100
+Connection ~ 2800 3100
+Connection ~ 2800 2500
 Wire Wire Line
-	3100 3700 3600 3700
-Connection ~ 3100 3700
-Wire Wire Line
-	3600 2550 4600 2550
-Wire Wire Line
-	3600 2550 3600 3100
-Connection ~ 3100 3100
-Wire Wire Line
-	3100 3100 3600 3100
-Connection ~ 3600 3100
-Wire Wire Line
-	3600 3100 3600 3250
-Wire Wire Line
-	3600 3700 3600 4200
-Wire Wire Line
-	3600 4200 4600 4200
-Connection ~ 3600 3700
+	2800 2500 3200 2500
 $Comp
 L Device:LED D1
@@
 P 5300 2900
 F 0 "R3" V 5093 2900 50  0000 C CNN
-F 1 "135" V 5184 2900 50  0000 C CNN
+F 1 "330" V 5184 2900 50  0000 C CNN
 F 2 "" V 5230 2900 50  0001 C CNN
 F 3 "~" H 5300 2900 50  0001 C CNN
@@
 	1    0    0    -1
 $EndComp
+Connection ~ 1900 3100
+Wire Wire Line
+	1900 3100 2800 3100
+$Comp
+L Device:C C3
+U 1 1 607D9F45
+P 3650 2800
+F 0 "C3" H 3765 2846 50  0000 L CNN
+F 1 "470 uF" H 3765 2755 50  0000 L CNN
+F 2 "" H 3688 2650 50  0001 C CNN
+F 3 "~" H 3650 2800 50  0001 C CNN
+	1    3650 2800
+	1    0    0    -1
+$EndComp
+Wire Wire Line
+	3200 2650 3200 2500
+Connection ~ 3200 2500
+Wire Wire Line
+	3200 2950 3200 3100
+Connection ~ 3200 3100
+Wire Wire Line
+	3650 3100 3650 2950
+Wire Wire Line
+	3200 3100 3650 3100
+Wire Wire Line
+	3650 2650 3650 2500
+Wire Wire Line
+	3200 2500 3650 2500
+Wire Wire Line
+	3650 2500 4100 2500
+Wire Wire Line
+	4600 2500 4600 2700
+Connection ~ 3650 2500
+Wire Wire Line
+	3650 3100 3650 4200
+Wire Wire Line
+	3650 4200 4600 4200
+Connection ~ 3650 3100
+Text Notes 4300 2250 0    50   ~ 0
+LED Voltage, V = 3.3 V\nLED Currect, I = 10 mA (brightness will be same, but LED life will be longer)\nResistor, R = U/I = 330 Om\n
+$Comp
+L Device:R R4
+U 1 1 60856124
+P 4100 2700
+F 0 "R4" H 4170 2746 50  0000 L CNN
+F 1 "100K" H 4170 2655 50  0000 L CNN
+F 2 "" V 4030 2700 50  0001 C CNN
+F 3 "~" H 4100 2700 50  0001 C CNN
+	1    4100 2700
+	1    0    0    -1
+$EndComp
+Wire Wire Line
+	4100 2900 4100 2850
+Wire Wire Line
+	4100 2550 4100 2500
+Connection ~ 4100 2500
+Wire Wire Line
+	4100 2500 4600 2500
 $EndSCHEMATC
