File: 2_Btn&Swtch.sch (KiCad schematic (older format))
At the start: 11 parts, among them SW1 Button, SW2 Switch

Commit message: All tasks were edited after feedback
Parts:
- removed DA1: AMS1117, Package_TO_SOT_SMD:SOT-223-3_TabPin2, symbol Regulator_Linear:AMS1117
- removed SW2: Switch, symbol Switch:SW_DIP_x01
- added 220K: R5, symbol Device:R
- added C4: 100 nF, symbol Device:C
- added DA?: AMS1117, Package_TO_SOT_SMD:SOT-223-3_TabPin2, symbol Regulator_Linear:AMS1117
- added R6: 100, symbol Device:R
- added R7: 100K, symbol Device:R
- added SW2: SW2, symbol Switch:SW_DPDT_x2
- C3: value 0.1uF -> 470 uF
- R1: value 124 -> 130
- R2: value 175 -> 180
- R3: value 1k -> 330
Connections:
- wire segments 33 -> 43
Other:
- moved on the sheet: R3, R4
