File: 4_Stabilization&LED&Btn.sch (KiCad schematic (older format))
At the start: 10 parts, among them SW1 Button, U1 LM317

Commit message: All tasks were edited after feedback
Parts:
- removed U1: LM317, Package_SO:SOIC-8_3.9x4.9mm_P1.27mm, symbol Regulator_Linear:LM317L_SO8
- added C1: 22 uF, symbol Device:CP1
- added C2: 10 uF, symbol Device:CP1
- added C3: 470 uF, symbol Device:C
- added DA1: AMS1117, Package_TO_SOT_SMD:SOT-223-3_TabPin2, symbol Regulator_Linear:AMS1117
- added R6: 220K, symbol Device:R
- added R6: 100K, symbol Device:R
- C4: renamed from C3; value 0.1 uF -> 100 nF
- R1: value 240 -> 130
- R2: value 2.4k -> 180
- R3: value 1k -> 100
- R4: value 135 -> 330
- R5: value 0.2 -> 330
Connections:
- net labels added: +3.3V, 7-12V, VDD
- net labels removed: +7-12V, VCC
- wire segments 15 -> 36
Other:
- moved on the sheet: C4
