File: 5_Potentiometer.sch (KiCad schematic (older format))
At the start: 6 parts, among them U1 LM317

Commit message: All tasks were edited after feedback
Parts:
- removed U1: LM317, Package_SO:SOIC-8_3.9x4.9mm_P1.27mm, symbol Regulator_Linear:LM317L_SO8
- added C1: 10 uF, symbol Device:CP1
- added C2: 22 uF, symbol Device:CP1
- added C3: 470 uF, symbol Device:C
- added DA1: AMS1117, Package_TO_SOT_SMD:SOT-223-3_TabPin2, symbol Regulator_Linear:AMS1117
- added R3: 100, symbol Device:R
- added R4: 1K, symbol Device:R
- R1: value 240 -> 130
- R2: value 2.4k -> 180
- R5: value 0.2 -> 100K
- RV1: value R_POT -> 10K
Connections:
- net labels added: +3.3V, +5V
- net labels removed: +7-12V, VCC
- wire segments 8 -> 31
Other:
- note added: "+3.3V\n"
- note removed: "3.3V\n"
