File: 9_BrushlessMotorControl.sch (KiCad schematic (older format))
At the start: 10 parts, among them M1 Aerodrive SK3 2826, U1 LM317, U2 SK3_2826

Commit message: All tasks were edited after feedback
Parts:
- removed BT? (x3): Battery_Cell, symbol Device:Battery_Cell
- removed M1: Aerodrive SK3 2826, symbol Motor:Stepper_Motor_unipolar_6pin
- removed U1: LM317, Package_SO:SOIC-8_3.9x4.9mm_P1.27mm, symbol Regulator_Linear:LM317L_SO8
- removed U2: SK3_2826, Package_SO:SOIC-8-1EP_3.9x4.9mm_P1.27mm_EP2.41x3.3mm, symbol Driver_Motor:SK3_2826
- added C1: 10 uF, symbol Device:CP1
- added C3: 22 uF, symbol Device:CP1
- added C4: 470 uF, symbol Device:C
- added DA1: AMS1117, Package_TO_SOT_SMD:SOT-223-3_TabPin2, symbol Regulator_Linear:AMS1117
- added M1: Motor_Servo, symbol Motor:Motor_Servo
- R1: value 240 -> 130
- R2: value 2.4k -> 180
- R3: value 0.2 -> 100K
Connections:
- net labels added: +3.3V, +5V
- net labels removed: +11.1V, B+, B-
- wire segments 40 -> 28
Other:
- note added: "PWM TIM1_Ch2\n\n"
- note removed: "PWM TIM3_Ch4\n"
