File: 13_BrushlessMotor&Batteries.sch (KiCad schematic (older format))
At the start: 9 parts, among them M1 Aerodrive SK3 2826, U1 LM317, U2 SK3_2826

Commit message: One more change
Parts:
- added R3: 100K, symbol Device:R
Connections:
- wire segments 24 -> 27
Changed lines of the file:
@@
 3.3V\n
 Wire Wire Line
-	3750 2450 4600 2450
+	3750 2450 4100 2450
 $Comp
 L Device:Battery_Cell BT?
@@
 	1    0    0    -1
 $EndComp
+$Comp
+L Device:R R3
+U 1 1 608397C4
+P 4100 2650
+F 0 "R3" H 4170 2696 50  0000 L CNN
+F 1 "100K" H 4170 2605 50  0000 L CNN
+F 2 "" V 4030 2650 50  0001 C CNN
+F 3 "~" H 4100 2650 50  0001 C CNN
+	1    4100 2650
+	1    0    0    -1
+$EndComp
+Wire Wire Line
+	4100 2500 4100 2450
+Connection ~ 4100 2450
+Wire Wire Line
+	4100 2450 4600 2450
+Wire Wire Line
+	4100 2800 4100 2900
 $EndSCHEMATC
